File: aerolotl_av.kicad_pcb (KiCad board)
At the start: 4 copper layers, 145.3 x 142.5 mm, 168 parts, among them J1 FTSH-107-STDC14, J10 GPIO_PE7-PE11, J11 USART3, J12 LPUART1, J13 WJ128V-5.0-2P, J14 WJ128V-5.0-2P, J2 Battery (ext.), J3 USB_C_Receptacle_USB2.0_16P, J4 SMA, J5 TF-102-15_SD_read, J6 I2C1, J7 I2C4, J8 I2C3, J9 GPIO_PE2-PE6, Q1 DMP2022LSS-13, Q2 AO3400A, Q3 AO3400A, Q4 AO3400A, Q5 DMP2022LSS-13, Q6 DMP2022LSS-13, SW1 SW_Push, SW2 SW_SPST, SW3 SW_SPST, U1 STM32G473VET6, U10 Ra-01H, U11 Airlift, U2 USBLC6-2P6, U3 TPS63802DLAR, U4 TPS2116DRL, U5 MAX-M10S, U6 BMP581, U7 BMI088, U8 ADXL345BCCZ-RL7, U9 ADXL375BCCZ-RL7, Y1 25MHz, Y2 32.768kHz

Commit message: most trace routing done
Parts:
- removed D3: STM LED, LED_SMD:LED_0805_2012Metric
- removed R23: 470, Resistor_SMD:R_0402_1005Metric
- D2: value RS-3535MWAR-2JYJY-J -> STATUS
- D4: value 3V3 LED -> 3V3
- D5: value USB LED -> USB
- D6: value ARM LED -> ARM
- D7: value LED red -> IGN0
- D8: value LED red -> IGN1
- F1, F2: footprint Fuse:Fuse_1812_4532Metric -> aerolotl_custom:Fuse_1812_4532Metric
- J1: value FTSH-107-STDC14 -> SWD
- J2: footprint Connector_AMASS:AMASS_XT30UPB-M_1x02_P5.0mm_Vertical -> aerolotl_custom:AMASS_XT30UPB-M_1x02_P5.0mm_Vertical
- J3: footprint Connector_USB:USB_C_Receptacle_HRO_TYPE-C-31-M-12 -> aerolotl_custom:USB_C_Receptacle_HRO_TYPE-C-31-M-12
- SW1: value SW_Push -> Reset
- SW2: value SW_SPST -> BOOT; footprint Button_Switch_SMD:SW_SPST_TL3342 -> aerolotl_custom:SW_DIP_SPSTx01_Kingtek_DSWB01LHGET_W7.62mm
- SW3: value SW_SPST -> ARM_SW
- TP1, TP10, TP11, TP2, TP3, TP4, TP7, TP8, TP9: footprint TestPoint:TestPoint_Plated_Hole_D2.0mm -> aerolotl_custom:TestPoint_KOA_RCTCTE_2.0x1.25mm
- TP5: value GND -> VSYS; footprint TestPoint:TestPoint_Plated_Hole_D2.0mm -> aerolotl_custom:TestPoint_KOA_RCTCTE_2.0x1.25mm
- TP6: footprint TestPoint:TestPoint_Pad_D1.5mm -> aerolotl_custom:TestPoint_KOA_RCTCTE_2.0x1.25mm
- U5: footprint RF_GPS:ublox_MAX -> aerolotl_custom:ublox_MAX
- U8: value ADXL345BCCZ-RL7 -> ADXL345
- U9: value ADXL375BCCZ-RL7 -> ADXL375
- moved J3 126.2 mm to (212.1, 107.7), turned to 90.1287 degrees
- moved R6 112.8 mm to (206.2, 105.2), turned to 90 degrees
- moved R5 112.2 mm to (205.9, 109.4), turned to 180 degrees
- moved J4 112.0 mm to (82.4, 108.6), turned to 90 degrees
- moved C18 111.5 mm to (204.6, 111.9), turned to -90 degrees
- moved U2 111.3 mm to (205.2, 107.6), turned to 180 degrees
- moved R7 105.8 mm to (201.6, 110.2), turned to 0 degrees
- moved C37 103.4 mm to (85.9, 114.0), turned to 180 degrees
- moved C38 103.2 mm to (87.4, 111.7), turned to 90 degrees
- moved C21 100.6 mm to (199.0, 112.8), turned to 180 degrees
- moved TP3 99.3 mm to (188.7, 83.4)
- moved R9 85.0 mm to (172.7, 82.8)
- moved R10 84.5 mm to (179.2, 82.9)
- moved U10 83.7 mm to (97.0, 115.7), turned to 0 degrees
- moved TP4 83.4 mm to (169.2, 82.5)
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Connections:
- net /Power/USB_DM renamed /Power/USB_D_M
- net /Power/USB_DP renamed /Power/USB_D_P
- TP5 pad 1: GND -> /Power/VSYS
- U1 pad 60: /Indicators/LED -> /MCU/MCU_LED
Routing:
- net GND: track 0.00 -> 227.1 mm, vias 303 -> 322
- net +3V3: track 0.00 -> 138.5 mm, vias 0 -> 36
- net +VBAT_ARM: track 0.00 -> 109.7 mm, vias 0 -> 2
- net /Igniter/IGN0: track 0.00 -> 99.8 mm, vias 0 -> 4
- net /External/I2C3.SCL: track 0.00 -> 99.2 mm, vias 0 -> 6
- net /MCU/RADIO_DIO4: track 0.00 -> 92.3 mm, vias 0 -> 2
- net /Igniter/SENSE_I0: track 0.00 -> 92.0 mm, vias 0 -> 4
- net /Power/VOLT_SENSE: track 0.00 -> 90.8 mm, vias 0 -> 6
- net /External/I2C4.SDA: track 0.00 -> 85.8 mm, vias 0 -> 6
- net /MCU/PWR_STS: track 0.00 -> 84.1 mm, vias 0 -> 2
- net /MCU/RADIO_RST: track 0.00 -> 83.6 mm, vias 0 -> 2
- net /External/GPIO.PE10: track 0.00 -> 83.4 mm, vias 0 -> 7
- net /Igniter/IGN1: track 0.00 -> 81.0 mm, vias 0 -> 4
- net /MCU/RADIO_DIO3: track 0.00 -> 80.4 mm, vias 0 -> 6
- net /MCU/RADIO_DIO0: track 0.00 -> 78.4 mm
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- added copper zone on F.Cu, net +3V3
- added copper zone on F.Cu, net /Power/P_VBUS
Other:
- board text added: "+x"
- board text added: "+y"
- board text added: "+z"
- board text added: "DROGUE (CH0)"
- board text added: "MAIN (CH1)"
- board text added: "ON"
- board text added: "diameter is 5.72 inches rn, hopefully everything fits"
- board text removed: "6 inch diameter. (might have to change circle diameter later w accordance to ID/OD)"
- board text removed: "BATT (bottom)"
- board text removed: "DROGUE (CH0) + -"
- board text removed: "DROGUE (J14 on bottom)"
- board text removed: "J10"
- board text removed: "J11"
- board text removed: "MAIN (CH1) + -"
- board text removed: "PLACE J4 (USB-C, after F8)"
