File: lora.kicad_sch (KiCad schematic)
At the start: 6 parts, among them J4 SMA, U10 Ra-01H

Commit message: most trace routing done
Parts:
- TP6: footprint TestPoint:TestPoint_Pad_D1.5mm -> aerolotl_custom:TestPoint_KOA_RCTCTE_2.0x1.25mm; LCSC Part (none) -> C172771; MPN (none) -> RCTCTE; Manufacturer (none) -> KOA Speer; now in the parts list
Changed lines of the file:
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@@
 		(body_style 1)
 		(exclude_from_sim no)
-		(in_bom no)
+		(in_bom yes)
 		(on_board yes)
 		(in_pos_files yes)
@@
 			)
 		)
-		(property "Footprint" "TestPoint:TestPoint_Pad_D1.5mm"
+		(property "Footprint" "aerolotl_custom:TestPoint_KOA_RCTCTE_2.0x1.25mm"
 			(at 109.22 72.39 0)
 			(hide yes)
@@
 			)
 		)
-		(property "Datasheet" ""
+		(property "Datasheet" "https://www.lcsc.com/datasheet/C172771.pdf"
 			(at 109.22 72.39 0)
 			(hide yes)
@@
 			(show_name no)
 			(do_not_autoplace no)
+			(effects
+				(font
+					(size 1.27 1.27)
+				)
+			)
+		)
+		(property "Manufacturer" "KOA Speer"
+			(at 109.22 72.39 0)
+			(hide yes)
+			(show_name no)
+			(do_not_autoplace no)
+			(effects
+				(font
+					(size 1.27 1.27)
+				)
+			)
+		)
+		(property "MPN" "RCTCTE"
+			(at 109.22 72.39 0)
+			(hide yes)
+			(show_name no)
+			(do_not_autoplace no)
+			(effects
+				(font
+					(size 1.27 1.27)
+				)
+			)
+		)
+		(property "LCSC Part" "C172771"
+			(at 109.22 72.39 0)
+			(hide yes)
+			(show_name no)
+			(do_not_autoplace no)
