File: sheets/igniter.kicad_sch (KiCad schematic)
At the start: 43 parts, among them J13 WJ128V-5.0-2P, J14 WJ128V-5.0-2P, Q3 AO3400A, Q4 AO3400A, Q5 DMP2022LSS-13, Q6 DMP2022LSS-13

Commit message: most trace routing done
Parts:
- D7: value LED red -> IGN0
- D8: value LED red -> IGN1
- F1, F2: footprint Fuse:Fuse_1812_4532Metric -> aerolotl_custom:Fuse_1812_4532Metric
- TP10, TP11, TP7, TP8, TP9: footprint TestPoint:TestPoint_Plated_Hole_D2.0mm -> aerolotl_custom:TestPoint_KOA_RCTCTE_2.0x1.25mm; LCSC Part (none) -> C172771; MPN (none) -> RCTCTE; Manufacturer (none) -> KOA Speer; now in the parts list
Changed lines of the file:
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@@
 			)
 		)
-		(property "Footprint" "Fuse:Fuse_1812_4532Metric"
+		(property "Footprint" "aerolotl_custom:Fuse_1812_4532Metric"
 			(at 97.79 100.33 0)
 			(hide yes)
@@
 		(body_style 1)
 		(exclude_from_sim no)
-		(in_bom no)
+		(in_bom yes)
 		(on_board yes)
 		(in_pos_files yes)
@@
 			)
 		)
-		(property "Footprint" "TestPoint:TestPoint_Plated_Hole_D2.0mm"
+		(property "Footprint" "aerolotl_custom:TestPoint_KOA_RCTCTE_2.0x1.25mm"
 			(at 228.6 82.55 0)
 			(hide yes)
@@
 			)
 		)
-		(property "Datasheet" ""
+		(property "Datasheet" "https://www.lcsc.com/datasheet/C172771.pdf"
 			(at 228.6 82.55 0)
 			(hide yes)
@@
 			)
 		)
+		(property "Manufacturer" "KOA Speer"
+			(at 228.6 82.55 0)
+			(hide yes)
+			(show_name no)
+			(do_not_autoplace no)
+			(effects
+				(font
+					(size 1.27 1.27)
+				)
+			)
+		)
+		(property "MPN" "RCTCTE"
+			(at 228.6 82.55 0)
+			(hide yes)
+			(show_name no)
+			(do_not_autoplace no)
+			(effects
+				(font
+					(size 1.27 1.27)
+				)
+			)
+		)
+		(property "LCSC Part" "C172771"
+			(at 228.6 82.55 0)
+			(hide yes)
+			(show_name no)
+			(do_not_autoplace no)
+			(effects
+				(font
+					(size 1.27 1.27)
+				)
+			)
+		)
 		(property "DCR" ""
 			(at 228.6 82.55 0)
@@
 		(body_style 1)
 		(exclude_from_sim no)
-		(in_bom no)
+		(in_bom yes)
 		(on_board yes)
 		(in_pos_files yes)
@@
 			)
 		)
-		(property "Footprint" "TestPoint:TestPoint_Plated_Hole_D2.0mm"
+		(property "Footprint" "aerolotl_custom:TestPoint_KOA_RCTCTE_2.0x1.25mm"
 			(at 228.6 36.83 0)
 			(hide yes)
@@
 			)
 		)
-		(property "Datasheet" ""
+		(property "Datasheet" "https://www.lcsc.com/datasheet/C172771.pdf"
 			(at 228.6 36.83 0)
 			(hide yes)
@@
 			)
 		)
+		(property "Manufacturer" "KOA Speer"
+			(at 228.6 36.83 0)
+			(hide yes)
+			(show_name no)
+			(do_not_autoplace no)
+			(effects
+				(font
+					(size 1.27 1.27)
+				)
+			)
+		)
+		(property "MPN" "RCTCTE"
+			(at 228.6 36.83 0)
+			(hide yes)
+			(show_name no)
+			(do_not_autoplace no)
+			(effects
+				(font
+					(size 1.27 1.27)
+				)
+			)
+		)
+		(property "LCSC Part" "C172771"
+			(at 228.6 36.83 0)
+			(hide yes)
+			(show_name no)
+			(do_not_autoplace no)
+			(effects
+				(font
+					(size 1.27 1.27)
+				)
+			)
+		)
 		(property "DCR" ""
 			(at 228.6 36.83 0)
@@
 			)
 		)
-		(property "Footprint" "Fuse:Fuse_1812_4532Metric"
+		(property "Footprint" "aerolotl_custom:Fuse_1812_4532Metric"
 			(at 101.6 194.31 0)
 			(hide yes)
@@
 			)
 		)
-		(property "Value" "LED red"
+		(property "Value" "IGN1"
 			(at 46.99 168.91 90)
-			(hide yes)
 			(show_name no)
 			(do_not_autoplace no)
@@
 		(body_style 1)
 		(exclude_from_sim no)
-		(in_bom no)
+		(in_bom yes)
 		(on_board yes)
 		(in_pos_files yes)
@@
 			)
 		)
-		(property "Footprint" "TestPoint:TestPoint_Plated_Hole_D2.0mm"
+		(property "Footprint" "aerolotl_custom:TestPoint_KOA_RCTCTE_2.0x1.25mm"
 			(at 228.6 97.79 0)
 			(hide yes)
@@
 			)
 		)
-		(property "Datasheet" ""
+		(property "Datasheet" "https://www.lcsc.com/datasheet/C172771.pdf"
 			(at 228.6 97.79 0)
 			(hide yes)
@@
 			)
 		)
+		(property "Manufacturer" "KOA Speer"
+			(at 228.6 97.79 0)
+			(hide yes)
+			(show_name no)
+			(do_not_autoplace no)
+			(effects
+				(font
+					(size 1.27 1.27)
+				)
+			)
+		)
+		(property "MPN" "RCTCTE"
+			(at 228.6 97.79 0)
+			(hide yes)
+			(show_name no)
+			(do_not_autoplace no)
+			(effects
+				(font
+					(size 1.27 1.27)
+				)
+			)
+		)
+		(property "LCSC Part" "C172771"
+			(at 228.6 97.79 0)
+			(hide yes)
+			(show_name no)
+			(do_not_autoplace no)
+			(effects
+				(font
+					(size 1.27 1.27)
+				)
+			)
+		)
 		(property "DCR" ""
 			(at 228.6 97.79 0)
@@
 		(body_style 1)
 		(exclude_from_sim no)
-		(in_bom no)
+		(in_bom yes)
 		(on_board yes)
 		(in_pos_files yes)
@@
 			)
 		)
-		(property "Footprint" "TestPoint:TestPoint_Plated_Hole_D2.0mm"
+		(property "Footprint" "aerolotl_custom:TestPoint_KOA_RCTCTE_2.0x1.25mm"
 			(at 228.6 67.31 0)
 			(hide yes)
@@
 			)
 		)
-		(property "Datasheet" ""
+		(property "Datasheet" "https://www.lcsc.com/datasheet/C172771.pdf"
 			(at 228.6 67.31 0)
 			(hide yes)
@@
 			)
 		)
+		(property "Manufacturer" "KOA Speer"
+			(at 228.6 67.31 0)
+			(hide yes)
+			(show_name no)
+			(do_not_autoplace no)
+			(effects
+				(font
+					(size 1.27 1.27)
+				)
+			)
+		)
+		(property "MPN" "RCTCTE"
+			(at 228.6 67.31 0)
+			(hide yes)
+			(show_name no)
+			(do_not_autoplace no)
+			(effects
+				(font
+					(size 1.27 1.27)
+				)
+			)
+		)
+		(property "LCSC Part" "C172771"
+			(at 228.6 67.31 0)
+			(hide yes)
+			(show_name no)
+			(do_not_autoplace no)
+			(effects
+				(font
+					(size 1.27 1.27)
+				)
+			)
+		)
 		(property "DCR" ""
 			(at 228.6 67.31 0)
@@
 			)
 		)
-		(property "Value" "LED red"
+		(property "Value" "IGN0"
 			(at 43.18 77.47 90)
-			(hide yes)
 			(show_name no)
 			(do_not_autoplace no)
@@
 		(body_style 1)
 		(exclude_from_sim no)
-		(in_bom no)
+		(in_bom yes)
 		(on_board yes)
 		(in_pos_files yes)
@@
 			)
 		)
-		(property "Footprint" "TestPoint:TestPoint_Plated_Hole_D2.0mm"
+		(property "Footprint" "aerolotl_custom:TestPoint_KOA_RCTCTE_2.0x1.25mm"
 			(at 228.6 52.07 0)
 			(hide yes)
@@
 			)
 		)
-		(property "Datasheet" ""
+		(property "Datasheet" "https://www.lcsc.com/datasheet/C172771.pdf"
 			(at 228.6 52.07 0)
 			(hide yes)
@@
 			(show_name no)
 			(do_not_autoplace no)
+			(effects
+				(font
+					(size 1.27 1.27)
+				)
+			)
+		)
+		(property "Manufacturer" "KOA Speer"
+			(at 228.6 52.07 0)
+			(hide yes)
+			(show_name no)
+			(do_not_autoplace no)
+			(effects
+				(font
+					(size 1.27 1.27)
+				)
+			)
+		)
+		(property "MPN" "RCTCTE"
+			(at 228.6 52.07 0)
+			(hide yes)
+			(show_name no)
+			(do_not_autoplace no)
+			(effects
+				(font
+					(size 1.27 1.27)
+				)
+			)
+		)
+		(property "LCSC Part" "C172771"
+			(at 228.6 52.07 0)
+			(hide yes)
+			(show_name no)
+			(do_not_autoplace no)
