File: sheets/power.kicad_sch (KiCad schematic)
At the start: 32 parts, among them J2 Battery (ext.), J3 USB_C_Receptacle_USB2.0_16P, Q1 DMP2022LSS-13, SW3 SW_SPST, U2 USBLC6-2P6, U3 TPS63802DLAR, U4 TPS2116DRL

Commit message: most trace routing done
Parts:
- J2: footprint Connector_AMASS:AMASS_XT30UPB-M_1x02_P5.0mm_Vertical -> aerolotl_custom:AMASS_XT30UPB-M_1x02_P5.0mm_Vertical
- J3: footprint Connector_USB:USB_C_Receptacle_HRO_TYPE-C-31-M-12 -> aerolotl_custom:USB_C_Receptacle_HRO_TYPE-C-31-M-12
- SW3: value SW_SPST -> ARM_SW
- TP1, TP2, TP3, TP4: footprint TestPoint:TestPoint_Plated_Hole_D2.0mm -> aerolotl_custom:TestPoint_KOA_RCTCTE_2.0x1.25mm; LCSC Part (none) -> C172771; MPN (none) -> RCTCTE; Manufacturer (none) -> KOA Speer; now in the parts list
- TP5: value GND -> VSYS; footprint TestPoint:TestPoint_Plated_Hole_D2.0mm -> aerolotl_custom:TestPoint_KOA_RCTCTE_2.0x1.25mm; LCSC Part (none) -> C172771; MPN (none) -> RCTCTE; Manufacturer (none) -> KOA Speer; now in the parts list
Connections:
- net GND: no longer TP5.1
- net VSYS: now also TP5.1
- net USB_DM renamed USB_D_M
- net USB_DP renamed USB_D_P
Other:
- moved on the sheet: R5, R6
