File: sheets/sensors.kicad_sch (KiCad schematic)
At the start: 20 parts, among them U5 MAX-M10S, U6 BMP581, U7 BMI088, U8 ADXL345BCCZ-RL7, U9 ADXL375BCCZ-RL7

Commit message: most trace routing done
Parts:
- U5: footprint RF_GPS:ublox_MAX -> aerolotl_custom:ublox_MAX
- U8: value ADXL345BCCZ-RL7 -> ADXL345
- U9: value ADXL375BCCZ-RL7 -> ADXL375
Changed lines of the file:
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@@
 			)
 		)
-		(property "Value" "ADXL345BCCZ-RL7"
+		(property "Value" "ADXL345"
 			(at 199.39 39.37 0)
 			(show_name no)
@@
 			)
 		)
-		(property "Value" "ADXL375BCCZ-RL7"
+		(property "Value" "ADXL375"
 			(at 204.47 133.35 0)
 			(show_name no)
@@
 			)
 		)
-		(property "Footprint" "RF_GPS:ublox_MAX"
+		(property "Footprint" "aerolotl_custom:ublox_MAX"
 			(at 76.2 135.89 0)
 			(hide yes)
