File: backups/aerolotl_av.pre_libfix.kicad_pcb (KiCad board)
At the start: 4 copper layers, 145.3 x 142.5 mm, 166 parts, among them J1 SWD, J10 GPIO_PE7-PE11, J11 USART3, J12 LPUART1, J13 WJ128V-5.0-2P, J14 WJ128V-5.0-2P, J2 Battery (ext.), J3 USB_C_Receptacle_USB2.0_16P, J4 SMA, J5 TF-102-15_SD_read, J6 I2C1, J7 I2C4, J8 I2C3, J9 GPIO_PE2-PE6, Q1 DMP2022LSS-13, Q2 AO3400A, Q3 AO3400A, Q4 AO3400A, Q5 DMP2022LSS-13, Q6 DMP2022LSS-13, SW1 Reset, SW2 BOOT, SW3 ARM_SW, U1 STM32G473VET6, U10 Ra-01H, U11 Airlift, U2 USBLC6-2P6, U3 TPS63802DLAR, U4 TPS2116DRL, U5 MAX-M10S, U6 BMP581, U7 BMI088, U8 ADXL345, U9 ADXL375, Y1 25MHz, Y2 32.768kHz

Commit message: all warnings and errors cleared. next step: order board
Parts:
- moved R5 0.13 mm to (205.9, 109.4)
